File: Level_shifter.kicad_sch (KiCad schematic)
At the start: 3 parts, among them Q4 SI2302S

Commit message: Start routing
Parts:
- renumbered Q4 to Q3, R44 to R42, R45 to R43
Changed lines of the file:
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@@
-(kicad_sch (version 20211123) (generator eeschema)
+(kicad_sch (version 20230121) (generator eeschema)
   (paper "A4")
   (junction (at 49.53 40.64) (diameter 0) (color 0 0 0 0)
@@
   )
   (wire (pts (xy 64.77 50.8) (xy 64.77 48.26))
-    (stroke (width 0) (type default) (color 0 0 0 0))
+    (stroke (width 0) (type default))
   )
   (wire (pts (xy 64.77 40.64) (xy 67.31 40.64))
-    (stroke (width 0) (type default) (color 0 0 0 0))
+    (stroke (width 0) (type default))
   )
   (wire (pts (xy 49.53 50.8) (xy 49.53 48.26))
-    (stroke (width 0) (type default) (color 0 0 0 0))
+    (stroke (width 0) (type default))
   )
   (wire (pts (xy 57.15 48.26) (xy 57.15 50.8))
-    (stroke (width 0) (type default) (color 0 0 0 0))
+    (stroke (width 0) (type default))
   )
   (wire (pts (xy 62.23 40.64) (xy 64.77 40.64))
-    (stroke (width 0) (type default) (color 0 0 0 0))
+    (stroke (width 0) (type default))
   )
   (wire (pts (xy 60.96 50.8) (xy 64.77 50.8))
-    (stroke (width 0) (type default) (color 0 0 0 0))
+    (stroke (width 0) (type default))
   )
   (wire (pts (xy 49.53 40.64) (xy 52.07 40.64))
-    (stroke (width 0) (type default) (color 0 0 0 0))
+    (stroke (width 0) (type default))
   )
   (wire (pts (xy 46.99 40.64) (xy 49.53 40.64))
-    (stroke (width 0) (type default) (color 0 0 0 0))
+    (stroke (width 0) (type default))
   )
   (wire (pts (xy 57.15 50.8) (xy 60.96 50.8))
-    (stroke (width 0) (type default) (color 0 0 0 0))
+    (stroke (width 0) (type default))
   )
-  (hierarchical_label "OUT" (shape output) (at 67.31 40.64 0)
+  (hierarchical_label "OUT" (shape output) (at 67.31 40.64 0) (fields_autoplaced)
     (effects (font (size 1.27 1.27)) (justify left))
   )
-  (hierarchical_label "IN" (shape input) (at 46.99 40.64 180)
+  (hierarchical_label "IN" (shape input) (at 46.99 40.64 180) (fields_autoplaced)
     (effects (font (size 1.27 1.27)) (justify right))
   )
-  (symbol (lib_id "Device:R") (at 49.53 44.45 0)
-    (in_bom yes) (on_board yes)
-    (property "Reference" "R44" (id 0) (at 51.308 43.2816 0)
+  (symbol (lib_id "Device:R") (at 49.53 44.45 0) (unit 1)
+    (in_bom yes) (on_board yes) (dnp no)
+    (property "Reference" "R42" (at 51.308 43.2816 0)
       (effects (font (size 1.27 1.27)) (justify left))
     )
-    (property "Value" "10k" (id 1) (at 51.308 45.593 0)
+    (property "Value" "10k" (at 51.308 45.593 0)
       (effects (font (size 1.27 1.27)) (justify left))
     )
-    (property "Footprint" "Resistor_SMD:R_0603_1608Metric" (id 2) (at 47.752 44.45 90)
+    (property "Footprint" "Resistor_SMD:R_0603_1608Metric" (at 47.752 44.45 90)
       (effects (font (size 1.27 1.27)) hide)
     )
-    (property "Datasheet" "~" (id 3) (at 49.53 44.45 0)
+    (property "Datasheet" "~" (at 49.53 44.45 0)
       (effects (font (size 1.27 1.27)) hide)
     )
     (pin "1")
     (pin "2")
+    (instances
+      (project "Tabac_Zynq"
+        (path "/e63e39d7-6ac0-4ffd-8aa3-1841a4541b55/f5ddbb84-39da-467f-99b8-af2beb2ad6ab"
+          (reference "R42") (unit 1)
+        )
+        (path "/e63e39d7-6ac0-4ffd-8aa3-1841a4541b55/631dd07b-c34d-40a1-ac32-ed7f4f5ac732"
+          (reference "R44") (unit 1)
+        )
+      )
+    )
   )
-  (symbol (lib_id "power:+5V") (at 60.96 50.8 180)
-    (in_bom yes) (on_board yes)
-    (property "Reference" "#PWR062" (id 0) (at 60.96 46.99 0)
+  (symbol (lib_id "power:+5V") (at 60.96 50.8 180) (unit 1)
+    (in_bom yes) (on_board yes) (dnp no)
+    (property "Reference" "#PWR060" (at 60.96 46.99 0)
       (effects (font (size 1.27 1.27)) hide)
     )
-    (property "Value" "+5V" (id 1) (at 62.23 54.61 0)
+    (property "Value" "+5V" (at 62.23 54.61 0)
       (effects (font (size 1.27 1.27)) (justify left))
     )
-    (property "Footprint" "" (id 2) (at 60.96 50.8 0)
+    (property "Footprint" "" (at 60.96 50.8 0)
       (effects (font (size 1.27 1.27)) hide)
     )
-    (property "Datasheet" "" (id 3) (at 60.96 50.8 0)
+    (property "Datasheet" "" (at 60.96 50.8 0)
       (effects (font (size 1.27 1.27)) hide)
     )
     (pin "1")
+    (instances
+      (project "Tabac_Zynq"
+        (path "/e63e39d7-6ac0-4ffd-8aa3-1841a4541b55/f5ddbb84-39da-467f-99b8-af2beb2ad6ab"
+          (reference "#PWR060") (unit 1)
+        )
+        (path "/e63e39d7-6ac0-4ffd-8aa3-1841a4541b55/631dd07b-c34d-40a1-ac32-ed7f4f5ac732"
+          (reference "#PWR062") (unit 1)
+        )
+      )
+    )
   )
-  (symbol (lib_id "Device:R") (at 64.77 44.45 0)
-    (in_bom yes) (on_board yes)
-    (property "Reference" "R45" (id 0) (at 66.548 43.2816 0)
+  (symbol (lib_id "Device:R") (at 64.77 44.45 0) (unit 1)
+    (in_bom yes) (on_board yes) (dnp no)
+    (property "Reference" "R43" (at 66.548 43.2816 0)
       (effects (font (size 1.27 1.27)) (justify left))
     )
-    (property "Value" "10k" (id 1) (at 66.548 45.593 0)
+    (property "Value" "10k" (at 66.548 45.593 0)
       (effects (font (size 1.27 1.27)) (justify left))
     )
-    (property "Footprint" "Resistor_SMD:R_0603_1608Metric" (id 2) (at 62.992 44.45 90)
+    (property "Footprint" "Resistor_SMD:R_0603_1608Metric" (at 62.992 44.45 90)
       (effects (font (size 1.27 1.27)) hide)
     )
-    (property "Datasheet" "~" (id 3) (at 64.77 44.45 0)
+    (property "Datasheet" "~" (at 64.77 44.45 0)
       (effects (font (size 1.27 1.27)) hide)
     )
     (pin "1")
     (pin "2")
+    (instances
+      (project "Tabac_Zynq"
+        (path "/e63e39d7-6ac0-4ffd-8aa3-1841a4541b55/f5ddbb84-39da-467f-99b8-af2beb2ad6ab"
+          (reference "R43") (unit 1)
+        )
+        (path "/e63e39d7-6ac0-4ffd-8aa3-1841a4541b55/631dd07b-c34d-40a1-ac32-ed7f4f5ac732"
+          (reference "R45") (unit 1)
+        )
+      )
+    )
   )
-  (symbol (lib_id "power:+3.3V") (at 49.53 50.8 180)
-    (in_bom yes) (on_board yes)
-    (property "Reference" "#PWR063" (id 0) (at 49.53 46.99 0)
+  (symbol (lib_id "power:+3.3V") (at 49.53 50.8 180) (unit 1)
+    (in_bom yes) (on_board yes) (dnp no)
+    (property "Reference" "#PWR061" (at 49.53 46.99 0)
       (effects (font (size 1.27 1.27)) hide)
     )
-    (property "Value" "+3.3V" (id 1) (at 49.53 54.61 0))
-    (property "Footprint" "" (id 2) (at 49.53 50.8 0)
+    (property "Value" "+3.3V" (at 49.53 54.61 0)
+      (effects (font (size 1.27 1.27)))
+    )
+    (property "Footprint" "" (at 49.53 50.8 0)
       (effects (font (size 1.27 1.27)) hide)
     )
-    (property "Datasheet" "" (id 3) (at 49.53 50.8 0)
+    (property "Datasheet" "" (at 49.53 50.8 0)
       (effects (font (size 1.27 1.27)) hide)
     )
     (pin "1")
+    (instances
+      (project "Tabac_Zynq"
+        (path "/e63e39d7-6ac0-4ffd-8aa3-1841a4541b55/f5ddbb84-39da-467f-99b8-af2beb2ad6ab"
+          (reference "#PWR061") (unit 1)
+        )
+        (path "/e63e39d7-6ac0-4ffd-8aa3-1841a4541b55/631dd07b-c34d-40a1-ac32-ed7f4f5ac732"
+          (reference "#PWR063") (unit 1)
+        )
+      )
+    )
   )
-  (symbol (lib_id "Device:Q_NMOS_GDS") (at 57.15 43.18 90)
-    (in_bom yes) (on_board yes)
-    (property "Reference" "Q4" (id 0) (at 57.15 34.4932 90))
-    (property "Value" "SI2302S" (id 1) (at 57.15 36.8046 90))
-    (property "Footprint" "Package_TO_SOT_SMD:SOT-23" (id 2) (at 54.61 38.1 0)
+  (symbol (lib_id "Device:Q_NMOS_GDS") (at 57.15 43.18 90) (unit 1)
+    (in_bom yes) (on_board yes) (dnp no)
+    (property "Reference" "Q3" (at 57.15 34.4932 90)
+      (effects (font (size 1.27 1.27)))
+    )
+    (property "Value" "SI2302S" (at 57.15 36.8046 90)
+      (effects (font (size 1.27 1.27)))
+    )
+    (property "Footprint" "Package_TO_SOT_SMD:SOT-23" (at 54.61 38.1 0)
       (effects (font (size 1.27 1.27)) hide)
     )
-    (property "Datasheet" "~" (id 3) (at 57.15 43.18 0)
+    (property "Datasheet" "~" (at 57.15 43.18 0)
       (effects (font (size 1.27 1.27)) hide)
     )
@@
     (pin "2")
     (pin "3")
+    (instances
+      (project "Tabac_Zynq"
+        (path "/e63e39d7-6ac0-4ffd-8aa3-1841a4541b55/f5ddbb84-39da-467f-99b8-af2beb2ad6ab"
+          (reference "Q3") (unit 1)
+        )
+        (path "/e63e39d7-6ac0-4ffd-8aa3-1841a4541b55/631dd07b-c34d-40a1-ac32-ed7f4f5ac732"
+          (reference "Q4") (unit 1)
+        )
+      )
+    )
   )
 )
