File: Tabac_Zynq.kicad_pcb (KiCad board)
At the start: 6 copper layers, 135 parts, among them IC1 S27KS0643GABHV020, J1 USB_C_Receptacle_USB2.0, J2 WSLED0, J3 WSLED1, J4 Conn_01x05_Male, Q1 MMBT2222ALT1G, Q2 MMBT2222ALT1G, Q3 SI2302S, Q4 SI2302S, SW1 RST, SW2 BOOT, U1 ESP32-WROOM-32, U2 CP2102N-A01-GQFN24, U3 MX25L6433FM2I-08G, U4 NCP1117-3.3_SOT223, U5 XC6210B182MR, U6 XC6210B122MR, U7 ICE40HX8K-CB132, X1 XO53

Commit message: Start routing
Parts:
- removed C29, C54: 10u, Capacitor_SMD:C_0805_2012Metric
- removed C31, C34, C36, C38, C39, C40, C41, C42, C43, C44, C45, C46, C47, C50, C51, C52, C53: 100n, Capacitor_SMD:C_0402_1005Metric
- removed C55, C56: 100n, Capacitor_SMD:C_0805_2012Metric
- U7: value ICE40HX8K-CB132 -> ICE40UP5K-SG48ITR; footprint AREA_lib_composant:IC_ICE40HX8K-CB132 -> Package_DFN_QFN:QFN-48-1EP_7x7mm_P0.5mm_EP5.6x5.6mm
- moved H1 146.5 mm to (115.3, 47.7)
- moved H2 146.5 mm to (115.3, 39.8)
- moved H4 146.5 mm to (123.3, 39.8)
- moved H5 146.5 mm to (131.2, 39.8)
- moved C4 130.8 mm to (67.6, 147.5), turned to -90 degrees
- moved R36 120.6 mm to (88.0, 144.5), turned to 90 degrees
- moved SW2 120.5 mm to (128.8, 176.8)
- moved D4 120.1 mm to (88.0, 147.8), turned to -90 degrees
- moved D3 116.3 mm to (86.0, 147.8), turned to -90 degrees
- moved R2 115.8 mm to (97.0, 142.2)
- moved R35 111.1 mm to (86.0, 144.5), turned to 90 degrees
- moved C3 110.8 mm to (73.1, 147.5), turned to 90 degrees
- moved R13 102.7 mm to (92.0, 135.6), turned to -90 degrees
- moved R4 101.1 mm to (75.6, 122.8), turned to 90 degrees
- moved J4 99.9 mm to (190.4, 52.5)
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Connections:
- C27 pad 2: Net-(C27-Pad2) -> GND
- C28 pad 2: Net-(C27-Pad2) -> GND
- C33 pad 1: +3V3 -> +2V5
Routing:
- net +1V2: track 0.00 -> 14.8 mm, vias 0 -> 3
- net /FPGA/QSPI_D3: track 0.00 -> 8.64 mm
- net /FPGA/FLASH_SDO: track 0.00 -> 8.59 mm
- net /FPGA/FLASH_SCK: track 0.00 -> 8.57 mm
- net GND: track 0.00 -> 8.20 mm, vias 0 -> 7
- net /FPGA/QSPI_D2: track 0.00 -> 7.09 mm
- net /FPGA/FLASH_SDI: track 0.00 -> 6.73 mm
- net /FPGA/FLASH_CS: track 0.00 -> 6.37 mm
- net /FPGA/16MHZ_CLOCK: track 0.00 -> 4.72 mm
- net +3V3: track 0.00 -> 4.26 mm, vias 0 -> 2
- net +1V8: track 0.00 -> 2.40 mm, vias 0 -> 1
- net +2V5: track 0.00 -> 2.24 mm, vias 0 -> 1
- net /FPGA/FPGA_RESET: track 0.00 -> 1.91 mm
- net Net-(D9-A): track 0.00 -> 1.81 mm

Commit message: last update
Parts:
- removed C1, C12, C20: 100n, Capacitor_SMD:C_0805_2012Metric
- removed C14, C15, C16, C17, C32, C33, C35, C37, C48, C49: 100n, Capacitor_SMD:C_0402_1005Metric
- removed C18, C19: 1u, Capacitor_SMD:C_0402_1005Metric
- removed C21, C22: 10u, Capacitor_SMD:C_0805_2012Metric
- removed D5: LED_1V8, LED_SMD:LED_0805_2012Metric
- removed D6: LED_1V2, LED_SMD:LED_0805_2012Metric
- removed D7: 1N4148, Diode_SMD:D_SOD-123
- removed D8, D9: LED, LED_SMD:LED_0805_2012Metric
- removed IC1: S27KS0643GABHV020, AREA_lib_composant:BGA24C100P5X5_600X800X100
- removed Q3, Q4: SI2302S, Package_TO_SOT_SMD:SOT-23
- removed R18, R19, R20, R21, R22, R23, R24, R25, R26, R27, R28, R29, R30, R31, R32, R33, R34: 33, Resistor_SMD:R_0603_1608Metric
- removed R37, R38, R39, R40: 560, Resistor_SMD:R_0603_1608Metric
- removed R41: 10K, Resistor_SMD:R_0603_1608Metric
- removed R42, R43, R44, R45: 10k, Resistor_SMD:R_0603_1608Metric
- removed SW2: BOOT, Button_Switch_SMD:SW_SPST_FSMSM
- removed U5: XC6210B182MR, Package_TO_SOT_SMD:SOT-23-5
- removed U6: XC6210B122MR, Package_TO_SOT_SMD:SOT-23-5
- removed U7: ICE40UP5K-SG48ITR, Package_DFN_QFN:QFN-48-1EP_7x7mm_P0.5mm_EP5.6x5.6mm
- removed X1: XO53, Oscillator:Oscillator_SMD_EuroQuartz_XO53-4Pin_5.0x3.2mm
- added C29: 100n, Capacitor_SMD:C_0805_2012Metric, F.Cu at (121.8, 110.8)
- added F1: 3A, AREA_lib_composant:FUSE_3557-2, F.Cu at (150.8, 148.5)
- added G***: LOGO, LOGO, B.Cu at (135.0, 97.2)
- added J5: WSLED0, Connector_PinSocket_2.54mm:PinSocket_1x04_P2.54mm_Vertical, F.Cu at (127.0, 126.3)
- C25: value 10u -> 1000u/16V; footprint Capacitor_SMD:C_0805_2012Metric -> Capacitor_SMD:CP_Elec_10x10.5
- C26: value 10u -> 100u/25V; footprint Capacitor_SMD:C_0805_2012Metric -> Capacitor_SMD:CP_Elec_6.3x7.7
- C27, C30: value 10u -> 1u
- C28: footprint Capacitor_SMD:C_0402_1005Metric -> Capacitor_SMD:C_0805_2012Metric
- J2: footprint Connector_Molex:Molex_KK-254_AE-6410-03A_1x03_P2.54mm_Vertical -> Connector_PinSocket_2.54mm:PinSocket_1x04_P2.54mm_Vertical
- J3: value WSLED1 -> WSLED0; footprint Connector_Molex:Molex_KK-254_AE-6410-03A_1x03_P2.54mm_Vertical -> Connector_PinSocket_2.54mm:PinSocket_1x04_P2.54mm_Vertical
- J4: value Conn_01x05_Male -> WSLED0; footprint Connector_Molex:Molex_KK-254_AE-6410-05A_1x05_P2.54mm_Vertical -> Connector_PinSocket_2.54mm:PinSocket_1x04_P2.54mm_Vertical
- R1, R10, R13, R14, R15, R16, R17, R2, R3, R35, R36, R5, R6, R7, R8, R9: footprint Resistor_SMD:R_0603_1608Metric -> Resistor_SMD:R_0805_2012Metric
- R11, R12, R4: value 33 -> 10K; footprint Resistor_SMD:R_0603_1608Metric -> Resistor_SMD:R_0805_2012Metric
- SW1: value RST -> SW_SPDT; footprint Button_Switch_SMD:SW_SPST_FSMSM -> Connector_JST:JST_PH_B3B-PH-K_1x03_P2.00mm_Vertical
- U3: value MX25L6433FM2I-08G -> SN74LVC1T45DBV; footprint Package_SO:SOP-8_3.9x4.9mm_P1.27mm -> Package_TO_SOT_SMD:SOT-23-6
- moved H1 118.2 mm to (159.0, 157.5)
- moved H2 117.8 mm to (114.0, 157.5)
- moved J4 83.6 mm to (132.7, 113.0), turned to 90 degrees
- moved R1 82.4 mm to (124.0, 99.0), turned to 0 degrees
- moved C5 82.3 mm to (124.0, 89.6), turned to 180 degrees
- moved C4 79.5 mm to (124.0, 91.6), turned to 180 degrees
- moved C2 76.6 mm to (124.0, 93.6), turned to 180 degrees
- moved R6 73.1 mm to (139.0, 110.0), turned to 180 degrees
- moved U1 72.6 mm to (136.5, 98.0), turned to 0 degrees
- moved SW1 71.8 mm to (160.5, 107.8), turned to -90 degrees
- moved C3 71.7 mm to (124.0, 97.1), turned to 0 degrees
- moved D3 59.9 mm to (145.0, 158.5)
- moved D4 59.9 mm to (147.0, 158.5)
- moved R35 59.9 mm to (145.0, 155.2)
- moved R36 59.9 mm to (147.0, 155.2)
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Connections:
- C25 pad 1: +1V8 -> +5V
- C26 pad 1: +1V2 -> +5V
- C27 pad 1: +1V2 -> +3V3
- C28 pad 1: +1V2 -> +3V3
- C30 pad 1: +1V2 -> +5V
- J1 pad A4: +5V -> Net-(F1-Pad1)
- J1 pad A9: +5V -> Net-(F1-Pad1)
- J1 pad B4: +5V -> Net-(F1-Pad1)
- J1 pad B9: +5V -> Net-(F1-Pad1)
- J2 pad 3: /Level_shifter/OUT -> /WSLED0_IN
- J3 pad 3: /Level_shifter1/OUT -> /WSLED1_IN
- J4 pad 1: GND -> +5V
- J4 pad 2: /MOSI -> GND
- J4 pad 3: /CLK -> /WSLED2_IN
- J4 pad 4: /CS -> /WSLED2_OUT
- R11 pad 1: /WSLED0 -> +3V3
- R11 pad 2: /FPGA/OUT_LED0 -> Net-(SW1-A)
- R12 pad 1: /WSLED1 -> Net-(SW1-C)
- R12 pad 2: /FPGA/OUT_LED1 -> GND
- R4 pad 1: Net-(U1-IO18) -> Net-(U3-DIR)
- R4 pad 2: SPI_SCK -> GND
- R5 pad 1: Net-(U1-IO19) -> /WSLED0_OUT
- R5 pad 2: SPI_MISO -> /WSLED1_IN
- R6 pad 1: Net-(U1-IO23) -> /WSLED1_OUT
- R6 pad 2: SPI_MOSI -> /WSLED2_IN
- R7 pad 1: Net-(U1-IO5) -> /WSLED2_OUT
- R7 pad 2: SPI_CS -> /WSLED3_IN
- SW1 pad 1: GND -> Net-(SW1-A)
- SW1 pad 2: /EN -> /Switch_ON/OFF
- U1 pad 13: unconnected-(U1-IO14-Pad13) -> /WSLED0
- U1 pad 23: unconnected-(U1-IO15-Pad23) -> /WSLED1
- U1 pad 24: unconnected-(U1-IO2-Pad24) -> /Switch_ON/OFF
- U1 pad 29: Net-(U1-IO5) -> unconnected-(U1-IO5-Pad29)
- U1 pad 30: Net-(U1-IO18) -> unconnected-(U1-IO18-Pad30)
- U1 pad 31: Net-(U1-IO19) -> unconnected-(U1-IO19-Pad31)
- U1 pad 37: Net-(U1-IO23) -> unconnected-(U1-IO23-Pad37)
- U3 pad 1: /CS -> +3V3
- U3 pad 2: /MISO -> GND
- U3 pad 3: /D2 -> /WSLED0
- U3 pad 4: GND -> /WSLED0_IN
- U3 pad 5: /SDO -> Net-(U3-DIR)
- U3 pad 6: /CLK -> +5V
Routing:
- net +3V3: track 4.26 -> 97.8 mm, vias 2 -> 10
- net /TX: track 0.00 -> 67.0 mm, vias 0 -> 2
- net /RX: track 0.00 -> 63.4 mm, vias 0 -> 2
- net /EN: track 0.00 -> 60.8 mm, vias 0 -> 2
- net /IO0: track 0.00 -> 59.6 mm, vias 0 -> 2
- net GND: track 8.20 -> 49.5 mm, vias 7 -> 98
- net /WSLED0_IN: track 0.00 -> 39.5 mm
- net +5V: track 0.00 -> 35.1 mm, vias 0 -> 16
- net /WSLED2_OUT: track 0.00 -> 21.1 mm
- net /WSLED1_OUT: track 0.00 -> 19.8 mm
- net /WSLED1_IN: track 0.00 -> 19.5 mm
- net /Switch_ON/OFF: track 0.00 -> 19.3 mm, vias 0 -> 1
- net /RTS: track 0.00 -> 16.0 mm
- net +1V2: track 14.8 -> 0.00 mm, vias 3 -> 0
- net /USB+: track 0.00 -> 13.8 mm
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- added copper zone on In2.Cu, net +3V3
- added copper zone on F.Cu, net +5V
- added copper zone on In2.Cu, net +5V
- added copper zone on B.Cu, net GND
- added copper zone on F.Cu, net GND
- added copper zone on In1.Cu, net GND
- added copper zone on In2.Cu, net GND
- added copper zone on In2.Cu, net Net-(F1-Pad1)
Other:
- board outline added: 51.5 x 76.5 mm
- copper layers 6 -> 4
- board text added: "3A"
- board text added: "3V3 5V"
- board text added: "5V"
- board text added: "DATA_IN"
- board text added: "DATA_OUT"
- board text added: "GND"
- board text added: "ON|OFF"
- board text added: "RX"
- board text added: "TX"
- board text added: "TX RX"
- board text added: "WLED Board Ptitcon Bière 2023 rev 1"
