File: Tabac_Zynq.kicad_sch (KiCad schematic)
At the start: 0 parts

Commit message: schematic finished
Parts:
- added C1, C11, C12, C13, C20, C3, C5: 100n, Capacitor_SMD:C_0805_2012Metric, symbol Device:C
- added C10, C2, C21, C22, C23, C24, C25, C26, C4, C8, C9: 10u, Capacitor_SMD:C_0805_2012Metric, symbol Device:C
- added C14, C15, C16, C17: 100n, Capacitor_SMD:C_0402_1005Metric, symbol Device:C
- added C18, C19: 1u, Capacitor_SMD:C_0402_1005Metric, symbol Device:C
- added C6, C7: 47p, Capacitor_SMD:C_0805_2012Metric, symbol Device:C
- added D1: LED_RX, LED_SMD:LED_0805_2012Metric, symbol Device:LED
- added D2: LED_TX, LED_SMD:LED_0805_2012Metric, symbol Device:LED
- added D3: LED_33V, LED_SMD:LED_0805_2012Metric, symbol Device:LED
- added D4: LED_5V, LED_SMD:LED_0805_2012Metric, symbol Device:LED
- added D5: LED_1V8, LED_SMD:LED_0805_2012Metric, symbol Device:LED
- added D6: LED_1V2, LED_SMD:LED_0805_2012Metric, symbol Device:LED
- added D7: 1N4148, Diode_SMD:D_SOD-123, symbol Diode:1N4148W
- added H1, H2, H4, H5: _, MountingHole:MountingHole_3.2mm_M3_Pad_Via, symbol Mechanical:MountingHole_Pad
- added IC1: S27KS0643GABHV020, AREA_lib_composant:BGA24C100P5X5_600X800X100, symbol AREA_composant:S27KS0643GABHV020
- added J1: USB_C_Receptacle_USB2.0, Connector_USB:USB_C_Receptacle_GCT_USB4085, symbol Connector:USB_C_Receptacle_USB2.0
- added J2: WSLED0, Connector_Molex:Molex_KK-254_AE-6410-03A_1x03_P2.54mm_Vertical, symbol Connector:Conn_01x03_Male
- added J3: WSLED1, Connector_Molex:Molex_KK-254_AE-6410-03A_1x03_P2.54mm_Vertical, symbol Connector:Conn_01x03_Male
- added J4: Conn_01x05_Male, Connector_Molex:Molex_KK-254_AE-6410-05A_1x05_P2.54mm_Vertical, symbol Connector:Conn_01x05_Male
- added Q1, Q2: MMBT2222ALT1G, Package_TO_SOT_SMD:SOT-23, symbol Device:Q_NPN_BEC
- added R1, R13, R14: 10K, Resistor_SMD:R_0603_1608Metric, symbol Device:R
- added R10: 10k, Resistor_SMD:R_0603_1608Metric, symbol Device:R
- added R11, R12, R18, R19, R20, R21, R22, R23, R24, R25, R26, R27, R28, R29, R30, R31, R32, R33, R34, R4, R5, R6, R7: 33, Resistor_SMD:R_0603_1608Metric, symbol Device:R
- added R15, R16, R35: 270, Resistor_SMD:R_0603_1608Metric, symbol Device:R
- added R17: 470, Resistor_SMD:R_0603_1608Metric, symbol Device:R
- added R2, R3: 5.1K, Resistor_SMD:R_0603_1608Metric, symbol Device:R
- added R36, R37, R38: 560, Resistor_SMD:R_0603_1608Metric, symbol Device:R
- added R8: 22k1, Resistor_SMD:R_0603_1608Metric, symbol Device:R
- added R9: 47k5, Resistor_SMD:R_0603_1608Metric, symbol Device:R
- added SW1: RST, Button_Switch_SMD:SW_SPST_FSMSM, symbol Switch:SW_Push
- added SW2: BOOT, Button_Switch_SMD:SW_SPST_FSMSM, symbol Switch:SW_Push
- added TP3: RX, TestPoint:TestPoint_Pad_D1.0mm, symbol Connector:TestPoint
- added TP4: TX, TestPoint:TestPoint_Pad_D1.0mm, symbol Connector:TestPoint
- added U1: ESP32-WROOM-32, RF_Module:ESP32-WROOM-32, symbol RF_Module:ESP32-WROOM-32
- added U2: CP2102N-A01-GQFN24, Package_DFN_QFN:QFN-24-1EP_4x4mm_P0.5mm_EP2.6x2.6mm, symbol Interface_USB:CP2102N-A01-GQFN24
- added U3: MX25L6433FM2I-08G, Package_SO:SOP-8_3.9x4.9mm_P1.27mm, symbol Memory_Flash:MX25R3235FM1xx0
- added U4: NCP1117-3.3_SOT223, Package_TO_SOT_SMD:SOT-223-3_TabPin2, symbol Regulator_Linear:NCP1117-3.3_SOT223
- added U5: XC6210B182MR, Package_TO_SOT_SMD:SOT-23-5, symbol Regulator_Linear:XC6210B332MR
- added U6: XC6210B122MR, Package_TO_SOT_SMD:SOT-23-5, symbol Regulator_Linear:XC6210B332MR
Connections:
- new net: D1.1 (K), R15.1
- new net: D6.1 (K), R38.1
- new net: R15.2, U2.13 (GPIO.1)
- new net: R17.2, U2.20 (RXD)
- new net: R7.1, U1.29 (IO5)
- new net: R4.1, U1.30 (IO18)
- new net: R5.1, U1.31 (IO19)
- new net: R6.1, U1.37 (IO23)
- new net: Q1.1 (B), R13.1
- new net: R8.2, R9.1, U2.8 (VBUS)
- new net: IC1.D2 (DQ1), R19.2
- new net: D5.1 (K), R37.1
- new net: Q2.1 (B), R14.1
- new net: IC1.C4 (DQ2), R20.2
- new net: IC1.D3 (DQ0), R18.2
- new net: IC1.D4 (DQ3), R21.2
- new net: IC1.D5 (DQ4), R22.2
- new net: IC1.E1 (DQ7), R25.2
- new net: IC1.E2 (DQ6), R24.2
- new net: IC1.E3 (DQ5), R23.2
- new net: R10.2, U2.9 (~{RSTb})
- new net: R16.2, U2.14 (GPIO.0)
- new net: D3.1 (K), R35.1
- new net: J1.B5 (CC2), R3.1
- new net: D4.1 (K), R36.1
- new net: J1.A5 (CC1), R2.2
- new net: D2.1 (K), R16.1
- new net +1V2: C26.1, D6.2 (A), U6.5 (VOUT)
- new net +1V8: C14.1, C15.1, C16.1, C17.1, C18.1, C19.1, C25.1, D5.2 (A), IC1.B4 (VCC), IC1.D1 (VCCQ_1), IC1.E4 (VCCQ_2), U5.5 (VOUT)
- new net +2V5: D7.1 (K)
- new net +3V3: C11.1, C2.1, C20.1, C24.1, C4.1, C5.1, C9.1, D1.2 (A), D2.2 (A), D3.2 (A), D7.2 (A), R1.1, R10.1, U1.2 (VDD), U2.6 (VDD), U2.7 (REGIN), U3.8 (VCC), U4.2 (VO)
- new net +5V: C10.1, C13.1, C21.1, C22.1, C23.1, C8.1, D4.2 (A), J1.A4 (VBUS), J1.A9 (VBUS), J1.B4 (VBUS), J1.B9 (VBUS), J2.1 (Pin_1), J3.1 (Pin_1), R8.1, U4.3 (VI), U5.1 (VIN), U5.3 (CE), U6.1 (VIN), U6.3 (CE)
- new net CLK: J4.3 (Pin_3), R30.2, U3.6 (SCLK)
- new net CS: J4.4 (Pin_4), R31.2, U3.1 (~{CS})
- new net D2: R32.2, U3.3 (~{WP}/SIO2)
- new net D3: R33.2, U3.7 (~{RESET}/SIO3)
- new net DTR: Q2.2 (E), R13.2, U2.23 (DTR)
- new net EN: C1.1, C3.2, Q1.3 (C), R1.2, SW1.2, U1.3 (EN)
- new net FPGA/FLASH_CS: R31.1
- new net FPGA/FLASH_SCK: R30.1
- new net FPGA/FLASH_SDI: R34.1
- new net FPGA/FLASH_SDO: R29.1
- new net FPGA/HYPERBUS_CLK+: IC1.B2 (CK)
- new net FPGA/HYPERBUS_CLK-: IC1.B1 (CK#)
- new net FPGA/HYPERBUS_CS#: R26.1
- new net FPGA/HYPERBUS_DQ0: R18.1
- new net FPGA/HYPERBUS_DQ1: R19.1
- new net FPGA/HYPERBUS_DQ2: R20.1
- new net FPGA/HYPERBUS_DQ3: R21.1
- new net FPGA/HYPERBUS_DQ4: R22.1
- new net FPGA/HYPERBUS_DQ5: R23.1
- new net FPGA/HYPERBUS_DQ6: R24.1
- new net FPGA/HYPERBUS_DQ7: R25.1
- new net FPGA/HYPERBUS_RESET#: R27.1
- new net FPGA/HYPERBUS_RWDS: R28.1
- new net FPGA/OUT_LED0: R11.2
- new net FPGA/OUT_LED1: R12.2
- new net FPGA/QSPI_D2: R32.1
- new net FPGA/QSPI_D3: R33.1
- new net GND: C1.2, C10.2, C11.2, C12.2, C13.2, C14.2, C15.2, C16.2, C17.2, C18.2, C19.2, C2.2, C20.2, C21.2, C22.2, C23.2, C24.2, C25.2, C26.2, C3.1, C4.2, C5.2, C6.2, C7.2, C8.2, C9.2, H1.1, H2.1, H4.1, H5.1, IC1.B3 (VSS), IC1.C1 (VSSQ_1), IC1.E5 (VSSQ_2), J1.A1 (GND), J1.A12 (GND), J1.B1 (GND), J1.B12 (GND), J1.S1 (SHIELD), J2.2 (Pin_2), J3.2 (Pin_2), J4.1 (Pin_1), R2.1, R3.2, R35.2, R36.2, R37.2, R38.2, R9.2, SW1.1, SW2.2, U1.1 (GND), U1.15 (GND), U1.38 (GND), U1.39 (GND), U2.2 (GND), U2.25 (GND), U3.4 (GND), U4.1 (GND), U5.2 (GND), U6.2 (GND)
- new net IO0: C12.1, Q2.3 (C), SW2.1, U1.25 (IO0)
- new net Level_shifter/OUT: J2.3 (Pin_3)
- new net Level_shifter1/OUT: J3.3 (Pin_3)
- new net MISO: J4.5 (Pin_5), R34.2, U3.2 (SO/SIO1)
- new net MOSI: J4.2 (Pin_2)
- new net RAM_CS#: IC1.A3 (CS#), R26.2
- new net RAM_RST#: IC1.A4 (RESET#), R27.2
- new net RAM_RWDS: IC1.C3 (RWDS), R28.2
- new net RTS: Q1.2 (E), R14.2, U2.19 (RTS)
- new net RX: R17.1, TP3.1, U1.35 (TXD0/IO1)
- new net SDO: R29.2, U3.5 (SI/SIO0)
- new net SPI_CS: R7.2
- new net SPI_MISO: R5.2
- new net SPI_MOSI: R6.2
- new net SPI_SCK: R4.2
- new net TX: TP4.1, U1.34 (RXD0/IO3), U2.21 (TXD)
- new net USB+: C6.1, J1.A6 (D+), J1.B6 (D+), U2.3 (D+)
- new net USB-: C7.1, J1.A7 (D-), J1.B7 (D-), U2.4 (D-)
- new net WSLED0: R11.1
- new net WSLED1: R12.1
- no-connect marks 0 -> 13
Other:
- removed sheet Peripheral
- removed sheet Power_regulation
- added sheet FPGA (FPGA.kicad_sch)
- added sheet Level_shifter (Level_shifter.kicad_sch)
- added sheet Level_shifter1 (Level_shifter.kicad_sch)
- note added: "Autoprogram"
- note added: "NC"
- note added: "Power supply 5V/3V3/1V2"
- note added: "USB to UART"

Commit message: Start routing
Parts:
- C12: now not fitted

Commit message: last update
Parts:
- removed C1, C12, C20: 100n, Capacitor_SMD:C_0805_2012Metric, symbol Device:C
- removed C14, C15, C16, C17: 100n, Capacitor_SMD:C_0402_1005Metric, symbol Device:C
- removed C18, C19: 1u, Capacitor_SMD:C_0402_1005Metric, symbol Device:C
- removed C21, C22, C25, C26: 10u, Capacitor_SMD:C_0805_2012Metric, symbol Device:C
- removed D5: LED_1V8, LED_SMD:LED_0805_2012Metric, symbol Device:LED
- removed D6: LED_1V2, LED_SMD:LED_0805_2012Metric, symbol Device:LED
- removed D7: 1N4148, Diode_SMD:D_SOD-123, symbol Diode:1N4148W
- removed IC1: S27KS0643GABHV020, AREA_lib_composant:BGA24C100P5X5_600X800X100, symbol AREA_composant:S27KS0643GABHV020
- removed J2: WSLED0, Connector_Molex:Molex_KK-254_AE-6410-03A_1x03_P2.54mm_Vertical, symbol Connector:Conn_01x03_Male
- removed J3: WSLED1, Connector_Molex:Molex_KK-254_AE-6410-03A_1x03_P2.54mm_Vertical, symbol Connector:Conn_01x03_Male
- removed J4: Conn_01x05_Male, Connector_Molex:Molex_KK-254_AE-6410-05A_1x05_P2.54mm_Vertical, symbol Connector:Conn_01x05_Male
- removed R18, R19, R20, R21, R22, R23, R24, R25, R26, R27, R28, R29, R30, R31, R32, R33, R34: 33, Resistor_SMD:R_0603_1608Metric, symbol Device:R
- removed R37, R38: 560, Resistor_SMD:R_0603_1608Metric, symbol Device:R
- removed SW1: RST, Button_Switch_SMD:SW_SPST_FSMSM, symbol Switch:SW_Push
- removed SW2: BOOT, Button_Switch_SMD:SW_SPST_FSMSM, symbol Switch:SW_Push
- removed U3: MX25L6433FM2I-08G, Package_SO:SOP-8_3.9x4.9mm_P1.27mm, symbol Memory_Flash:MX25R3235FM1xx0
- removed U5: XC6210B182MR, Package_TO_SOT_SMD:SOT-23-5, symbol Regulator_Linear:XC6210B332MR
- removed U6: XC6210B122MR, Package_TO_SOT_SMD:SOT-23-5, symbol Regulator_Linear:XC6210B332MR
- added C25: 1000u/16V, Capacitor_SMD:CP_Elec_10x10.5, symbol Device:C_Polarized_Small
- added C26: 100u/25V, Capacitor_SMD:CP_Elec_6.3x7.7, symbol Device:C_Polarized_Small
- added C27, C30: 1u, Capacitor_SMD:C_0805_2012Metric, symbol Device:C
- added C28, C29: 100n, Capacitor_SMD:C_0805_2012Metric, symbol Device:C
- added F1: 3A, AREA_lib_composant:FUSE_3557-2, symbol Device:Fuse
- added J2, J3, J4, J5: WSLED0, Connector_PinSocket_2.54mm:PinSocket_1x04_P2.54mm_Vertical, symbol Connector:Conn_01x04_Pin
- added SW1: SW_SPDT, Connector_JST:JST_PH_B3B-PH-K_1x03_P2.00mm_Vertical, symbol Switch:SW_SPDT
- added U3: SN74LVC1T45DBV, Package_TO_SOT_SMD:SOT-23-6, symbol Logic_LevelTranslator:SN74LVC1T45DBV
- C10, C8: now not fitted
- R1, R10, R13, R14, R15, R16, R17, R2, R3, R35, R36, R5, R6, R7, R8, R9: footprint Resistor_SMD:R_0603_1608Metric -> Resistor_SMD:R_0805_2012Metric
- R11, R12, R4: value 33 -> 10K; footprint Resistor_SMD:R_0603_1608Metric -> Resistor_SMD:R_0805_2012Metric
Connections:
- net FPGA/OUT_LED1 is gone; now on net GND: R12.2
- net SPI_SCK is gone; now on net GND: R4.2
- net +3V3: now also R11.1, C27.1, C28.1, U3.1 (VCCA)
- net +5V: now also C25.1, C26.1, C29.1, C30.1, F1.2, J2.1 (Pin_1), J3.1 (Pin_1), J4.1 (Pin_1), J5.1 (Pin_1), U3.6 (VCCB); no longer J1.A4 (VBUS), J1.A9 (VBUS), J1.B4 (VBUS), J1.B9 (VBUS)
- net GND: now also C25.2, C26.2, C27.2, C28.2, C29.2, C30.2, J2.2 (Pin_2), J3.2 (Pin_2), J4.2 (Pin_2), J5.2 (Pin_2), U3.2 (GND)
- net WSLED0: now also U1.13 (IO14), U3.3 (A); no longer R11.1
- net WSLED1: now also U1.23 (IO15); no longer R12.1
- net Switch_ON/OFF: now reaches U1.24 (IO2)
- net Switch_ON/OFF: now also SW1.2 (B)
- net at U1.29 (IO5): no longer R7.1
- net at R4.1: now also U3.5 (DIR); no longer U1.30 (IO18)
- net at U1.31 (IO19): no longer R5.1
- net at U1.37 (IO23): no longer R6.1
- net FPGA/OUT_LED0: no longer names the net of R11.2
- net FPGA/OUT_LED0: now also SW1.1 (A)
- net SPI_CS renamed WSLED3_IN
- net WSLED3_IN: now also J5.3 (Pin_3)
- net SPI_MISO renamed WSLED1_IN
- net WSLED1_IN: now also J3.3 (Pin_3)
- net SPI_MOSI renamed WSLED2_IN
- net WSLED2_IN: now also J4.3 (Pin_3)
- new net: F1.1, J1.A4 (VBUS), J1.A9 (VBUS), J1.B4 (VBUS), J1.B9 (VBUS)
- new net: R12.1, SW1.3 (C)
- new net WSLED0_IN: J2.3 (Pin_3), U3.4 (B)
- new net WSLED0_OUT: J2.4 (Pin_4), R5.1
- new net WSLED1_OUT: J3.4 (Pin_4), R6.1
- new net WSLED2_OUT: J4.4 (Pin_4), R7.1
- new net WSLED3_OUT: J5.4 (Pin_4)
- no-connect marks 13 -> 11
Other:
- removed sheet FPGA
- removed sheet Level_shifter
- removed sheet Level_shifter1
- note removed: "NC"
